File: hardware/buddy_main/audio_camera.kicad_sch (KiCad schematic)
At the start: 0 parts

Commit message: pcb build
Parts:
- added C31: 10uF 10V, Capacitor_SMD:C_0805_2012Metric, symbol Device:C
- added C32, C33, C36: 100nF, Capacitor_SMD:C_0603_1608Metric, symbol Device:C
- added C34, C35, C37: 1uF, Capacitor_SMD:C_0603_1608Metric, symbol Device:C
- added J10: CAMERA OV2640 24P, Connector_FFC-FPC:Hirose_FH12-24S-0.5SH_1x24-1MP_P0.50mm_Horizontal, symbol Connector_Generic_MountingPin:Conn_01x24_MountingPin
- added J8: SPEAKER 4-8R, Connector_JST:JST_PH_B2B-PH-K_1x02_P2.00mm_Vertical, symbol Connector_Generic:Conn_01x02
- added J9: I2S MIC (INMP441), Connector_PinSocket_2.54mm:PinSocket_1x06_P2.54mm_Vertical, symbol Connector_Generic:Conn_01x06
- added R18: 1M, Resistor_SMD:R_0603_1608Metric, symbol Device:R
- added R19, R20: 10k, Resistor_SMD:R_0603_1608Metric, symbol Device:R
- added R21, R22: 4.7k, Resistor_SMD:R_0603_1608Metric, symbol Device:R
- added U10: MAX98357A, Package_DFN_QFN:TQFN-16-1EP_3x3mm_P0.5mm_EP1.23x1.23mm, symbol Audio:MAX98357A
Connections:
- new net 1V2: C35.1, J10.10 (Pin_10)
- new net 2V8: C34.1, J10.4 (Pin_4)
- new net 3V3: C33.1, C37.1, J10.11 (Pin_11), J9.1 (Pin_1), R19.1, R21.1, R22.1
- new net 5V: C31.1, C32.1, R18.1, U10.7 (VDD), U10.8 (VDD)
- new net AMP_SD_MODE: R18.2, U10.4 (~{SD_MODE})
- new net CAM_HREF: J10.9 (Pin_9)
- new net CAM_PCLK: J10.17 (Pin_17)
- new net CAM_PWDN: J10.8 (Pin_8), R20.1
- new net CAM_RESET: C36.1, J10.6 (Pin_6), R19.2
- new net CAM_SIOC: J10.5 (Pin_5), R21.2
- new net CAM_SIOD: J10.3 (Pin_3), R22.2
- new net CAM_VSYNC: J10.7 (Pin_7)
- new net CAM_XCLK: J10.13 (Pin_13)
- new net CAM_Y2: J10.19 (Pin_19)
- new net CAM_Y3: J10.21 (Pin_21)
- new net CAM_Y4: J10.22 (Pin_22)
- new net CAM_Y5: J10.20 (Pin_20)
- new net CAM_Y6: J10.18 (Pin_18)
- new net CAM_Y7: J10.16 (Pin_16)
- new net CAM_Y8: J10.14 (Pin_14)
- new net CAM_Y9: J10.12 (Pin_12)
- new net GND: C31.2, C32.2, C33.2, C34.2, C35.2, C36.2, C37.2, J10.15 (Pin_15), J10.2 (Pin_2), J10.MP (MountPin), J9.2 (Pin_2), J9.6 (Pin_6), R20.2, U10.11 (GND), U10.15 (GND), U10.17 (PAD), U10.2 (GAIN_SLOT), U10.3 (GND)
- new net I2S_BCLK: J9.5 (Pin_5), U10.16 (BCLK)
- new net I2S_DIN: J9.3 (Pin_3)
- new net I2S_DOUT: U10.1 (DIN)
- new net I2S_WS: J9.4 (Pin_4), U10.14 (LRCLK)
- new net SPK_N: J8.2 (Pin_2), U10.10 (OUTN)
- new net SPK_P: J8.1 (Pin_1), U10.9 (OUTP)
- no-connect marks 0 -> 3
