File: hardware/buddy_main/mcu.kicad_sch (KiCad schematic)
At the start: 0 parts

Commit message: pcb build
Parts:
- added C18: 22uF 10V, Capacitor_SMD:C_0805_2012Metric, symbol Device:C
- added C19, C20: 100nF, Capacitor_SMD:C_0603_1608Metric, symbol Device:C
- added C21: 1uF, Capacitor_SMD:C_0603_1608Metric, symbol Device:C
- added D5: STATUS blue, LED_SMD:LED_0603_1608Metric, symbol Device:LED
- added J3: USB-C, Connector_USB:USB_C_Receptacle_GCT_USB4105-xx-A_16P_TopMnt_Horizontal, symbol Connector:USB_C_Receptacle_USB2.0_16P
- added J4: UART DEBUG, Connector_PinHeader_2.54mm:PinHeader_1x04_P2.54mm_Vertical, symbol Connector_Generic:Conn_01x04
- added R10, R11: 5.1k, Resistor_SMD:R_0603_1608Metric, symbol Device:R
- added R12: 1k, Resistor_SMD:R_0603_1608Metric, symbol Device:R
- added R8, R9: 10k, Resistor_SMD:R_0603_1608Metric, symbol Device:R
- added SW2: RESET, Button_Switch_SMD:SW_SPST_PTS810, symbol Switch:SW_Push
- added SW3: BOOT, Button_Switch_SMD:SW_SPST_PTS810, symbol Switch:SW_Push
- added U6: ESP32-S3-WROOM-1-N16R8, RF_Module:ESP32-S3-WROOM-1, symbol RF_Module:ESP32-S3-WROOM-1
- added U7: USBLC6-2SC6, Package_TO_SOT_SMD:SOT-23-6, symbol Power_Protection:USBLC6-2SC6
Connections:
- new net 3V3: C18.1, C19.1, C20.1, J4.4 (Pin_4), R8.1, R9.1, U6.2 (3V3)
- new net BOOT: R9.2, SW3.1, U6.27 (IO0)
- new net CAM_HREF: U6.7 (IO7)
- new net CAM_PCLK: U6.21 (IO13)
- new net CAM_SIOC: U6.5 (IO5)
- new net CAM_SIOD: U6.4 (IO4)
- new net CAM_VSYNC: U6.6 (IO6)
- new net CAM_XCLK: U6.8 (IO15)
- new net CAM_Y2: U6.19 (IO11)
- new net CAM_Y3: U6.17 (IO9)
- new net CAM_Y4: U6.12 (IO8)
- new net CAM_Y5: U6.18 (IO10)
- new net CAM_Y6: U6.20 (IO12)
- new net CAM_Y7: U6.11 (IO18)
- new net CAM_Y8: U6.10 (IO17)
- new net CAM_Y9: U6.9 (IO16)
- new net CC1: J3.A5 (CC1), R10.1
- new net CC2: J3.B5 (CC2), R11.1
- new net EN: C21.1, R8.2, SW2.1, U6.3 (EN)
- new net GND: C18.2, C19.2, C20.2, C21.2, D5.1 (K), J3.A1 (GND), J3.A12 (GND), J3.B1 (GND), J3.B12 (GND), J3.SH (SHIELD), J4.1 (Pin_1), R10.2, R11.2, SW2.2, SW3.2, U6.1 (GND), U6.40 (GND), U6.41 (GND), U7.2 (GND)
- new net I2S_BCLK: U6.34 (IO41)
- new net I2S_DIN: U6.32 (IO39)
- new net I2S_DOUT: U6.33 (IO40)
- new net I2S_WS: U6.35 (IO42)
- new net LED_STAT: R12.1, U6.16 (IO46)
- new net LED_STAT_A: D5.2 (A), R12.2
- new net M1_IN1: U6.38 (IO2)
- new net M1_IN2: U6.22 (IO14)
- new net M2_IN1: U6.23 (IO21)
- new net M2_IN2: U6.31 (IO38)
- new net M3_IN1: U6.24 (IO47)
- new net M3_IN2: U6.25 (IO48)
- new net MOT_nFAULT: U6.15 (IO3)
- new net MOT_nSLEEP: U6.26 (IO45)
- new net UART_RX: J4.3 (Pin_3), U6.36 (RXD0)
- new net UART_TX: J4.2 (Pin_2), U6.37 (TXD0)
- new net USB_DN: J3.A7 (D-), J3.B7 (D-), U6.13 (USB_D-), U7.3 (I/O2), U7.4 (I/O2)
- new net USB_DP: J3.A6 (D+), J3.B6 (D+), U6.14 (USB_D+), U7.1 (I/O1), U7.6 (I/O1)
- new net VBAT_SENSE: U6.39 (IO1)
- new net VBUS: J3.A4 (VBUS), J3.A9 (VBUS), J3.B4 (VBUS), J3.B9 (VBUS), U7.5 (VBUS)
- no-connect marks 0 -> 5
