File: hardware/buddy_main/motors.kicad_sch (KiCad schematic)
At the start: 0 parts

Commit message: pcb build
Parts:
- added C22, C26: 10uF 25V, Capacitor_SMD:C_1206_3216Metric, symbol Device:C
- added C23, C27: 100nF, Capacitor_SMD:C_0603_1608Metric, symbol Device:C
- added C24, C28: 10nF 16V, Capacitor_SMD:C_0603_1608Metric, symbol Device:C
- added C25, C29: 2.2uF, Capacitor_SMD:C_0603_1608Metric, symbol Device:C
- added C30: 47uF 16V, Capacitor_SMD:CP_Elec_6.3x7.7, symbol Device:C_Polarized
- added J5: MOTOR 1, Connector_JST:JST_XH_B2B-XH-A_1x02_P2.50mm_Vertical, symbol Connector_Generic:Conn_01x02
- added J6: MOTOR 2, Connector_JST:JST_XH_B2B-XH-A_1x02_P2.50mm_Vertical, symbol Connector_Generic:Conn_01x02
- added J7: MOTOR 3, Connector_JST:JST_XH_B2B-XH-A_1x02_P2.50mm_Vertical, symbol Connector_Generic:Conn_01x02
- added R13: 100k, Resistor_SMD:R_0603_1608Metric, symbol Device:R
- added R14: 10k, Resistor_SMD:R_0603_1608Metric, symbol Device:R
- added R15, R16, R17: 0.1R 1206, Resistor_SMD:R_1206_3216Metric, symbol Device:R
- added U8, U9: DRV8833PWP, Package_SO:HTSSOP-16-1EP_4.4x5mm_P0.65mm_EP3.4x5mm_Mask2.46x2.31mm_ThermalVias, symbol Driver_Motor:DRV8833PWP
Connections:
- new net 3V3: R14.2
- new net AISEN1: R15.1, U8.3 (AISEN)
- new net AISEN2: R17.1, U9.3 (AISEN)
- new net BISEN1: R16.1, U8.6 (BISEN)
- new net GND: C22.2, C23.2, C25.2, C26.2, C27.2, C29.2, C30.2, R13.2, R15.2, R16.2, R17.2, U8.13 (GND), U8.17 (GND), U9.10 (BIN2), U9.13 (GND), U9.17 (GND), U9.6 (BISEN), U9.9 (BIN1)
- new net M1_A: J5.1 (Pin_1), U8.2 (AOUT1)
- new net M1_B: J5.2 (Pin_2), U8.4 (AOUT2)
- new net M1_IN1: U8.16 (AIN1)
- new net M1_IN2: U8.15 (AIN2)
- new net M2_A: J6.1 (Pin_1), U8.7 (BOUT1)
- new net M2_B: J6.2 (Pin_2), U8.5 (BOUT2)
- new net M2_IN1: U8.9 (BIN1)
- new net M2_IN2: U8.10 (BIN2)
- new net M3_A: J7.1 (Pin_1), U9.2 (AOUT1)
- new net M3_B: J7.2 (Pin_2), U9.4 (AOUT2)
- new net M3_IN1: U9.16 (AIN1)
- new net M3_IN2: U9.15 (AIN2)
- new net MOT_nFAULT: R14.1, U8.8 (~{FAULT}), U9.8 (~{FAULT})
- new net MOT_nSLEEP: R13.1, U8.1 (~{SLEEP}), U9.1 (~{SLEEP})
- new net VCP1: C24.1, U8.11 (VCP)
- new net VCP2: C28.1, U9.11 (VCP)
- new net VINT1: C25.1, U8.14 (VINT)
- new net VINT2: C29.1, U9.14 (VINT)
- new net VSYS: C22.1, C23.1, C24.2, C26.1, C27.1, C28.2, C30.1, U8.12 (VM), U9.12 (VM)
- no-connect marks 0 -> 2
