File: hardware/buddy_main/power.kicad_sch (KiCad schematic)
At the start: 0 parts

Commit message: pcb build
Parts:
- added C1: 100uF 16V, Capacitor_SMD:CP_Elec_6.3x7.7, symbol Device:C_Polarized
- added C10, C11, C3, C5, C6: 100nF, Capacitor_SMD:C_0603_1608Metric, symbol Device:C
- added C12, C13, C7, C8: 22uF 10V, Capacitor_SMD:C_0805_2012Metric, symbol Device:C
- added C14, C15, C16, C17: 1uF, Capacitor_SMD:C_0603_1608Metric, symbol Device:C
- added C2, C4, C9: 10uF 25V, Capacitor_SMD:C_1206_3216Metric, symbol Device:C
- added D1: SMBJ24CA, Diode_SMD:D_SMB, symbol Device:D_TVS
- added D2: SMAJ5.0A, Diode_SMD:D_SMA, symbol Device:D_Zener
- added D3: SS34, Diode_SMD:D_SMA, symbol Device:D_Schottky
- added D4: PWR green, LED_SMD:LED_0603_1608Metric, symbol Device:LED
- added F1: PTC 3A hold, Fuse:Fuse_2920_7451Metric, symbol Device:Polyfuse
- added F2: PTC 1.1A hold, Fuse:Fuse_1206_3216Metric, symbol Device:Polyfuse
- added J1: XT30 BATTERY, Connector_AMASS:AMASS_XT30U-M_1x02_P5.0mm_Vertical, symbol Connector_Generic:Conn_01x02
- added J2: JST-PH BATTERY, Connector_JST:JST_PH_B2B-PH-K_1x02_P2.00mm_Vertical, symbol Connector_Generic:Conn_01x02
- added L1: 4.7uH, Inductor_SMD:L_Bourns_SRN6045TA, symbol Device:L
- added L2: 6.8uH, Inductor_SMD:L_Bourns_SRN6045TA, symbol Device:L
- added Q1: Si4214DDY, Package_SO:SOIC-8_3.9x4.9mm_P1.27mm, symbol Transistor_FET:Q_Dual_NMOS_S1G1S2G2D2D2D1D1
- added R1: 1M, Resistor_SMD:R_0603_1608Metric, symbol Device:R
- added R2, R6: 33k, Resistor_SMD:R_0603_1608Metric, symbol Device:R
- added R3: 56k, Resistor_SMD:R_0603_1608Metric, symbol Device:R
- added R4, R5: 100k, Resistor_SMD:R_0603_1608Metric, symbol Device:R
- added R7: 1k, Resistor_SMD:R_0603_1608Metric, symbol Device:R
- added SW1: POWER, Button_Switch_SMD:SW_SPDT_PCM12, symbol Switch:SW_SPDT
- added U1: LTC4365TS8, Package_TO_SOT_SMD:TSOT-23-8, symbol Power_Management:LTC4365TS8
- added U2: AP63203WU, Package_TO_SOT_SMD:TSOT-23-6, symbol Regulator_Switching:AP63203WU
- added U3: AP63205WU, Package_TO_SOT_SMD:TSOT-23-6, symbol Regulator_Switching:AP63205WU
- added U4: XC6206P282MR, Package_TO_SOT_SMD:SOT-23-3, symbol Regulator_Linear:XC6206PxxxMR
- added U5: XC6206P122MR, Package_TO_SOT_SMD:SOT-23-3, symbol Regulator_Linear:XC6206PxxxMR
Connections:
- new net 1V2: C17.1, U5.2 (VO)
- new net 2V8: C15.1, U4.2 (VO)
- new net 3V3: C14.1, C16.1, C7.1, C8.1, L1.2, R7.1, U2.1 (FB), U4.3 (VI), U5.3 (VI)
- new net 5V: C12.1, C13.1, L2.2, U3.1 (FB)
- new net BST_3V3: C6.1, U2.6 (BST)
- new net BST_5V: C11.1, U3.6 (BST)
- new net GATE: Q1.2 (G), Q1.4 (G), U1.8 (GATE)
- new net GND: C1.2, C10.2, C12.2, C13.2, C14.2, C15.2, C16.2, C17.2, C2.2, C3.2, C4.2, C5.2, C7.2, C8.2, C9.2, D1.2 (A2), D2.2 (A), D4.1 (K), J1.2 (Pin_2), J2.2 (Pin_2), R3.2, R6.2, SW1.1 (A), U1.4 (GND), U2.4 (GND), U3.4 (GND), U4.1 (GND), U5.1 (GND)
- new net LED_PWR: D4.2 (A), R7.2
- new net OV: R1.2, R2.1, U1.3 (OV)
- new net Q_SRC: Q1.1 (S), Q1.3 (S)
- new net SW_3V3: C6.2, L1.1, U2.5 (SW)
- new net SW_5V: C11.2, L2.1, U3.5 (SW)
- new net UV: R2.2, R3.1, U1.2 (UV)
- new net VBAT_F: D1.1 (A1), F1.2, Q1.7 (D), Q1.8 (D), R1.1, R4.1, U1.1 (Vin)
- new net VBAT_IN: F1.1, J1.1 (Pin_1), J2.1 (Pin_1)
- new net VBAT_SENSE: C3.1, R5.2, R6.1
- new net VBUS: F2.1
- new net VBUS_F: D2.1 (K), D3.2 (A), F2.2
- new net VSYS: C1.1, C10.1, C2.1, C4.1, C5.1, C9.1, D3.1 (K), Q1.5 (D), Q1.6 (D), R5.1, U1.7 (Vout), U2.2 (EN), U2.3 (IN), U3.2 (EN), U3.3 (IN)
- new net ~{SHDN}: R4.2, SW1.2 (B), U1.5 (~{SHDN})
- no-connect marks 0 -> 2
Other:
- note added: "BATTERY INPUT PROTECTION (2S LiPo / 6xAA) LTC4365 + back-to-back NMOS: reverse to -40V, OV trip 9.7V, UV trip 6.1V F1 3A PTC: short / stall protection. D1 bidirectional TVS: spikes only. SW1 = power switch (pulls ~SHDN low = OFF, carries uA only)"
- note added: "BUCK REGULATORS from VSYS (4.6-9.7V) U2 AP63203: 3V3 2A (ESP32, logic) U3 AP63205: 5V 2A (speaker amp)"
- note added: "CAMERA LDOs from 3V3: 2V8 (AVDD) and 1V2 (DVDD)"
- note added: "USB-C 5V INPUT: 1.1A PTC (protects the host port), 5V TVS, SS34 Schottky stops the battery back-feeding the USB host"
- note added: "VSYS SENSE -> ESP32 ADC (GPIO1) 100k/33k: 9.7V -> 2.4V"
