File: hardware/buddy_main/buddy_main.kicad_pcb (KiCad board)
At the start: 2 copper layers, 0 parts

Commit message: pcb build
Parts:
- added C1: 100uF 16V, Capacitor_SMD:CP_Elec_6.3x7.7, F.Cu at (111.0, 137.2)
- added C10: 100nF, Capacitor_SMD:C_0603_1608Metric, F.Cu at (132.5, 131.5)
- added C11: 100nF, Capacitor_SMD:C_0603_1608Metric, F.Cu at (132.5, 133.3)
- added C12: 22uF 10V, Capacitor_SMD:C_0805_2012Metric, F.Cu at (125.0, 134.5)
- added C13: 22uF 10V, Capacitor_SMD:C_0805_2012Metric, F.Cu at (128.8, 134.5)
- added C14: 1uF, Capacitor_SMD:C_0603_1608Metric, F.Cu at (124.5, 142.5)
- added C15: 1uF, Capacitor_SMD:C_0603_1608Metric, F.Cu at (124.5, 144.3)
- added C16: 1uF, Capacitor_SMD:C_0603_1608Metric, F.Cu at (129.5, 142.5)
- added C17: 1uF, Capacitor_SMD:C_0603_1608Metric, F.Cu at (129.5, 144.3)
- added C18: 22uF 10V, Capacitor_SMD:C_0805_2012Metric, F.Cu at (120.5, 104.0)
- added C19: 100nF, Capacitor_SMD:C_0603_1608Metric, F.Cu at (118.2, 104.3)
- added C2: 10uF 25V, Capacitor_SMD:C_1206_3216Metric, F.Cu at (120.6, 132.5)
- added C20: 100nF, Capacitor_SMD:C_0603_1608Metric, F.Cu at (141.5, 122.6)
- added C21: 1uF, Capacitor_SMD:C_0603_1608Metric, F.Cu at (139.5, 122.6)
- added C22: 10uF 25V, Capacitor_SMD:C_1206_3216Metric, F.Cu at (154.4, 110.7)
- added C23: 100nF, Capacitor_SMD:C_0603_1608Metric, F.Cu at (154.4, 113.2)
- added C24: 10nF 16V, Capacitor_SMD:C_0603_1608Metric, F.Cu at (144.0, 104.0)
- added C25: 2.2uF, Capacitor_SMD:C_0603_1608Metric, F.Cu at (144.0, 107.5)
- added C26: 10uF 25V, Capacitor_SMD:C_1206_3216Metric, F.Cu at (154.4, 121.6)
- added C27: 100nF, Capacitor_SMD:C_0603_1608Metric, F.Cu at (154.4, 124.2)
- added C28: 10nF 16V, Capacitor_SMD:C_0603_1608Metric, F.Cu at (144.0, 118.5)
- added C29: 2.2uF, Capacitor_SMD:C_0603_1608Metric, F.Cu at (144.0, 122.0)
- added C3: 100nF, Capacitor_SMD:C_0603_1608Metric, F.Cu at (117.5, 135.0)
- added C30: 47uF 16V, Capacitor_SMD:CP_Elec_6.3x7.7, F.Cu at (150.0, 131.5)
- added C31: 10uF 10V, Capacitor_SMD:C_0805_2012Metric, F.Cu at (150.0, 144.5)
- added C32: 100nF, Capacitor_SMD:C_0603_1608Metric, F.Cu at (145.0, 139.0)
- added C33: 100nF, Capacitor_SMD:C_0603_1608Metric, F.Cu at (154.5, 146.0)
- added C34: 1uF, Capacitor_SMD:C_0603_1608Metric, F.Cu at (138.0, 139.3)
- added C35: 1uF, Capacitor_SMD:C_0603_1608Metric, F.Cu at (141.5, 139.3)
- added C36: 100nF, Capacitor_SMD:C_0603_1608Metric, F.Cu at (134.5, 141.1)
- added C37: 1uF, Capacitor_SMD:C_0603_1608Metric, F.Cu at (138.0, 141.1)
- added C4: 10uF 25V, Capacitor_SMD:C_1206_3216Metric, F.Cu at (120.6, 127.8)
- added C5: 100nF, Capacitor_SMD:C_0603_1608Metric, F.Cu at (117.0, 131.0)
- added C6: 100nF, Capacitor_SMD:C_0603_1608Metric, F.Cu at (117.0, 132.8)
- added C7: 22uF 10V, Capacitor_SMD:C_0805_2012Metric, F.Cu at (103.2, 132.0)
- added C8: 22uF 10V, Capacitor_SMD:C_0805_2012Metric, F.Cu at (103.2, 134.4)
- added C9: 10uF 25V, Capacitor_SMD:C_1206_3216Metric, F.Cu at (136.6, 128.2)
- added D1: SMBJ24CA, Diode_SMD:D_SMB, F.Cu at (112.0, 116.2)
- added D2: SMAJ5.0A, Diode_SMD:D_SMA, F.Cu at (111.0, 143.0)
- added D3: SS34, Diode_SMD:D_SMA, F.Cu at (120.3, 140.0)
- added D4: PWR green, LED_SMD:LED_0603_1608Metric, F.Cu at (120.5, 111.6)
- added D5: STATUS blue, LED_SMD:LED_0603_1608Metric, F.Cu at (136.6, 134.3)
- added F1: PTC 3A hold, Fuse:Fuse_2920_7451Metric, F.Cu at (112.6, 110.0)
- added F2: PTC 1.1A hold, Fuse:Fuse_1206_3216Metric, F.Cu at (117.2, 141.5)
- added H1: MountingHole_2.7mm, MountingHole:MountingHole_2.7mm, F.Cu at (103.5, 103.5)
- added H2: MountingHole_2.7mm, MountingHole:MountingHole_2.7mm, F.Cu at (160.5, 103.5)
- added H3: MountingHole_2.7mm, MountingHole:MountingHole_2.7mm, F.Cu at (103.5, 152.5)
- added H4: MountingHole_2.7mm, MountingHole:MountingHole_2.7mm, F.Cu at (160.5, 152.5)
- added J1: XT30 BATTERY, Connector_AMASS:AMASS_XT30U-M_1x02_P5.0mm_Vertical, F.Cu at (103.5, 115.5)
- added J10: CAMERA OV2640 24P, Connector_FFC-FPC:Hirose_FH12-24S-0.5SH_1x24-1MP_P0.50mm_Horizontal, F.Cu at (131.5, 151.1)
- added J2: JST-PH BATTERY, Connector_JST:JST_PH_B2B-PH-K_1x02_P2.00mm_Vertical, F.Cu at (102.6, 126.5)
- added J3: USB-C, Connector_USB:USB_C_Receptacle_GCT_USB4105-xx-A_16P_TopMnt_Horizontal, F.Cu at (112.0, 151.8)
- added J4: UART DEBUG, Connector_PinHeader_2.54mm:PinHeader_1x04_P2.54mm_Vertical, F.Cu at (140.2, 126.6)
- added J5: MOTOR 1, Connector_JST:JST_XH_B2B-XH-A_1x02_P2.50mm_Vertical, F.Cu at (159.9, 112.5)
- added J6: MOTOR 2, Connector_JST:JST_XH_B2B-XH-A_1x02_P2.50mm_Vertical, F.Cu at (159.9, 121.0)
- added J7: MOTOR 3, Connector_JST:JST_XH_B2B-XH-A_1x02_P2.50mm_Vertical, F.Cu at (159.9, 129.5)
- added J8: SPEAKER 4-8R, Connector_JST:JST_PH_B2B-PH-K_1x02_P2.00mm_Vertical, F.Cu at (160.4, 140.5)
- added J9: I2S MIC (INMP441), Connector_PinSocket_2.54mm:PinSocket_1x06_P2.54mm_Vertical, F.Cu at (142.5, 153.4)
- added L1: 4.7uH, Inductor_SMD:L_Bourns_SRN6045TA, F.Cu at (110.5, 129.5)
- added L2: 6.8uH, Inductor_SMD:L_Bourns_SRN6045TA, F.Cu at (126.0, 129.0)
- added Q1: Si4214DDY, Package_SO:SOIC-8_3.9x4.9mm_P1.27mm, F.Cu at (112.0, 122.0)
- added R1: 1M, Resistor_SMD:R_0603_1608Metric, F.Cu at (118.2, 108.3)
- added R10: 5.1k, Resistor_SMD:R_0603_1608Metric, F.Cu at (119.0, 147.5)
- added R11: 5.1k, Resistor_SMD:R_0603_1608Metric, F.Cu at (121.0, 147.5)
- added R12: 1k, Resistor_SMD:R_0603_1608Metric, F.Cu at (136.6, 132.5)
- added R13: 100k, Resistor_SMD:R_0603_1608Metric, F.Cu at (144.0, 111.0)
- added R14: 10k, Resistor_SMD:R_0603_1608Metric, F.Cu at (144.0, 114.5)
- added R15: 0.1R 1206, Resistor_SMD:R_1206_3216Metric, F.Cu at (154.4, 104.5)
- added R16: 0.1R 1206, Resistor_SMD:R_1206_3216Metric, F.Cu at (154.4, 107.6)
- added R17: 0.1R 1206, Resistor_SMD:R_1206_3216Metric, F.Cu at (154.4, 118.5)
- added R18: 1M, Resistor_SMD:R_0603_1608Metric, F.Cu at (145.0, 142.6)
- added R19: 10k, Resistor_SMD:R_0603_1608Metric, F.Cu at (134.5, 137.5)
- added R2: 33k, Resistor_SMD:R_0603_1608Metric, F.Cu at (118.2, 111.6)
- added R20: 10k, Resistor_SMD:R_0603_1608Metric, F.Cu at (138.0, 137.5)
- added R21: 4.7k, Resistor_SMD:R_0603_1608Metric, F.Cu at (141.5, 137.5)
- added R22: 4.7k, Resistor_SMD:R_0603_1608Metric, F.Cu at (134.5, 139.3)
- added R3: 56k, Resistor_SMD:R_0603_1608Metric, F.Cu at (118.2, 114.9)
- added R4: 100k, Resistor_SMD:R_0603_1608Metric, F.Cu at (118.2, 118.2)
- added R5: 100k, Resistor_SMD:R_0603_1608Metric, F.Cu at (120.5, 114.9)
- added R6: 33k, Resistor_SMD:R_0603_1608Metric, F.Cu at (120.5, 118.2)
- added R7: 1k, Resistor_SMD:R_0603_1608Metric, F.Cu at (120.5, 108.3)
- added R8: 10k, Resistor_SMD:R_0603_1608Metric, F.Cu at (135.5, 122.6)
- added R9: 10k, Resistor_SMD:R_0603_1608Metric, F.Cu at (137.5, 122.6)
- added SW1: POWER, Button_Switch_SMD:SW_SPDT_PCM12, F.Cu at (112.5, 103.7)
- added SW2: RESET, Button_Switch_SMD:SW_SPST_PTS810, F.Cu at (125.3, 122.6)
- added SW3: BOOT, Button_Switch_SMD:SW_SPST_PTS810, F.Cu at (131.3, 122.6)
- added U1: LTC4365TS8, Package_TO_SOT_SMD:TSOT-23-8, F.Cu at (119.5, 122.0)
- added U10: MAX98357A, Package_DFN_QFN:TQFN-16-1EP_3x3mm_P0.5mm_EP1.23x1.23mm, F.Cu at (150.0, 140.0)
- added U2: AP63203WU, Package_TO_SOT_SMD:TSOT-23-6, F.Cu at (117.0, 127.5)
- added U3: AP63205WU, Package_TO_SOT_SMD:TSOT-23-6, F.Cu at (132.5, 128.0)
- added U4: XC6206P282MR, Package_TO_SOT_SMD:SOT-23-3, F.Cu at (125.0, 139.0)
- added U5: XC6206P122MR, Package_TO_SOT_SMD:SOT-23-3, F.Cu at (130.0, 139.0)
- added U6: ESP32-S3-WROOM-1-N16R8, RF_Module:ESP32-S3-WROOM-1, F.Cu at (132.0, 106.8)
- added U7: USBLC6-2SC6, Package_TO_SOT_SMD:SOT-23-6, F.Cu at (104.0, 142.0)
- added U8: DRV8833PWP, Package_SO:HTSSOP-16-1EP_4.4x5mm_P0.65mm_EP3.4x5mm_Mask2.46x2.31mm_ThermalVias, F.Cu at (149.0, 108.0)
- added U9: DRV8833PWP, Package_SO:HTSSOP-16-1EP_4.4x5mm_P0.65mm_EP3.4x5mm_Mask2.46x2.31mm_ThermalVias, F.Cu at (149.0, 122.0)
Other:
- board outline added: 64 x 56 mm

Commit message: fuh ton of routing
Other:
- copper layers 2 -> 4
Changed lines of the file:
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@@
 		(35 "F.Fab" user)
 		(33 "B.Fab" user)
+		(4 "In1.Cu" power)
+		(6 "In2.Cu" power)
 	)
 	(setup
